Commit message: rviz update

File: linorobot2/linorobot2_description/urdf/mech/base.urdf.xacro (robot description, xacro)
@@ -5,5 +5,5 @@
     <link name="base_link">
       <visual>
-        <origin xyz="0.02 -0.095 0" rpy="0 0 3.14"/>
+        <origin xyz="0 0 0" rpy="0 0 3.14"/>
         <geometry>
           <mesh scale="0.002 0.002 0.002" filename="file:///home/samet/Desktop/isaac-gym/base_link_centered.stl"/>
@@ -15,5 +15,5 @@
       </visual>
       <collision>
-        <origin xyz="0.02 -0.095 0" rpy="0 0 3.14"/>
+        <origin xyz="0 0 0" rpy="0 0 3.14"/>
         <geometry>
           <box size="${length} ${width} ${height}"/>

File: linorobot2/linorobot2_description/urdf/mech/mecanum_wheel.urdf.xacro (robot description, xacro)
@@ -4,5 +4,5 @@
     <link name="${side}_wheel_link">
       <visual>
-        <origin xyz="0 0 0" rpy="${pi/2} 0 0"/>
+        <origin xyz="0 0.1 0" rpy="${pi/2} 0 0"/>
         <geometry>
           <mesh scale="0.002 0.002 0.002" filename="file:///home/samet/Desktop/robomaster-stl-files/Robomaster_Sim/miror.stl"/>
@@ -27,6 +27,6 @@
     </link>
     <gazebo reference="${side}_wheel_link">
-        <mu1>0.01</mu1>
-        <mu2>0.01</mu2>
+        <mu1>0.1</mu1>
+        <mu2>0.1</mu2>
     </gazebo>
     <gazebo reference="${side}_wheel_link">

File: linorobot2/linorobot2_description/urdf/sensors/depth_sensor.urdf.xacro (robot description, xacro)
@@ -4,5 +4,5 @@
     <link name="camera_link">
       <visual>
-        <origin xyz="0 0 0" rpy="0 0 0"/>
+        <origin xyz="0 0.1 0" rpy="0 0 0"/>
         <geometry>
           <box size="0.030 0.124 0.030"/>

Commit message: little update

File: linorobot2/linorobot2_description/urdf/mech/base.urdf.xacro (robot description, xacro)
@@ -5,5 +5,5 @@
     <link name="base_link">
       <visual>
-        <origin xyz="0 0 0" rpy="0 0 3.14"/>
+        <origin xyz="0.02 0 0" rpy="0 0 3.14"/>
         <geometry>
           <mesh scale="0.002 0.002 0.002" filename="file:///home/samet/Desktop/isaac-gym/base_link_centered.stl"/>

File: linorobot2/linorobot2_description/urdf/mech/mecanum_wheel2.urdf.xacro (robot description, xacro)
@@ -1,10 +1,10 @@
 <?xml version="1.0"?>
 <robot xmlns:xacro="http://ros.org/wiki/xacro">
-  <xacro:macro name="mecanum_wheel" params="side radius width pos_x pos_y pos_z mass">
+  <xacro:macro name="mecanum_wheel2" params="side radius width pos_x pos_y pos_z mass">
     <link name="${side}_wheel_link">
       <visual>
-        <origin xyz="0 0.1 0" rpy="${pi/2} 0 0"/>
+        <origin xyz="0 0.21 0" rpy="${pi/2} 0 0"/>
         <geometry>
-          <mesh scale="0.002 0.002 0.002" filename="file:///home/samet/Desktop/robomaster-stl-files/Robomaster_Sim/miror.stl"/>
+          <mesh scale="0.002 0.002 0.002" filename="file:///home/samet/Desktop/robomaster-stl-files/Robomaster_Sim/Wheel_L.stl"/>
         </geometry>
         <material name="blue">

File: linorobot2/linorobot2_description/urdf/robots/mecanum.urdf.xacro (robot description, xacro)
@@ -4,4 +4,5 @@
   <xacro:include filename="$(find linorobot2_description)/urdf/mech/base.urdf.xacro" />
   <xacro:include filename="$(find linorobot2_description)/urdf/mech/mecanum_wheel.urdf.xacro" />
+  <xacro:include filename="$(find linorobot2_description)/urdf/mech/mecanum_wheel2.urdf.xacro" />
   <xacro:include filename="$(find linorobot2_description)/urdf/sensors/imu.urdf.xacro" />
   <xacro:include filename="$(find linorobot2_description)/urdf/sensors/generic_laser.urdf.xacro" />
@@ -16,5 +17,5 @@
     wheel_pos_z="${wheel_pos_z}"
 />
-  <xacro:mecanum_wheel
+  <xacro:mecanum_wheel2
     side="front_left"
     radius="${wheel_radius}"
@@ -43,5 +44,5 @@
     mass="${wheel_mass}"
   />
-  <xacro:mecanum_wheel
+  <xacro:mecanum_wheel2
     side="rear_right"
     radius="${wheel_radius}"

Commit message: add lidar and camera stl

File: linorobot2/linorobot2_description/urdf/mech/base.urdf.xacro (robot description, xacro)
@@ -28,4 +28,48 @@
       </inertial>
     </link>
+    <link name="rplidar">
+      <inertial>
+        <origin xyz="0 0 0" rpy="0 0 0"/>
+        <mass value="1"/>
+        <inertia ixx="0.1"  ixy="0"  ixz="0" iyy="0.1" iyz="0" izz="0.1" />
+      </inertial>
+      <visual>
+        <origin xyz="0 0 0" rpy="0 0 0" />
+        <geometry>
+          <mesh scale="0.002 0.002 0.002" filename="file:///home/samet/Desktop/robomaster-stl-files/Robomaster_Sim/lidar.stl"/>
+        </geometry>
+        <material name="yellow">
+          <color rgba="0.8784 0.6627 0.6627 1.0"/>
+        </material>
+      </visual>
+      <collision>
+        <origin xyz="0 0 0" rpy="0 0 0"/>
+        <geometry>
+          <box size="0.1 0.1 0.1" />
+        </geometry>
+      </collision>
+    </link>
+        <link name="camerafpv">
+      <inertial>
+        <origin xyz="0 0 0" rpy="0 0 0"/>
+        <mass value="1"/>
+        <inertia ixx="0.1"  ixy="0"  ixz="0" iyy="0.1" iyz="0" izz="0.1" />
+      </inertial>
+      <visual>
+        <origin xyz="0 0 0" rpy="0 0 0" />
+        <geometry>
+          <mesh scale="0.002 0.002 0.002" filename="file:///home/samet/Desktop/robomaster-stl-files/Robomaster_Sim/camera.stl"/>
+        </geometry>
+        <material name="yellow">
+          <color rgba="0.8784 0.6627 0.6627 1.0"/>
+        </material>
+      </visual>
+      <collision>
+        <origin xyz="0 0 0" rpy="0 0 0"/>
+        <geometry>
+          <box size="0.1 0.1 0.1" />
+        </geometry>
+      </collision>
+    </link>
     <gazebo reference="base_link">
       <visual>
@@ -43,4 +87,14 @@
       <origin xyz="0 0 ${wheel_radius - wheel_pos_z}" rpy="0 0 0"/>
     </joint>
+        <joint name="lidar_joint" type="fixed">
+      <parent link="base_link"/>
+      <child link="rplidar"/>
+      <origin xyz="0.05 0.015 0.29" rpy="0 0 1.57"/>
+    </joint>
+        <joint name="camera_joint" type="fixed">
+      <parent link="base_link"/>
+      <child link="camerafpv"/>
+      <origin xyz="0.2 0.04 0.12" rpy="1.57 0 1.57"/>
+    </joint>
   </xacro:macro>
 </robot>
